Commit message: Fully working

File: urdf/olv-lbracket.urdf.xacro (robot description, xacro)
@@ -12,7 +12,7 @@
     <xacro:if value="${mounting_side == 'top'}">
       <xacro:property name="body_translation" value="0 0.055 -0.024" />
-      <xacro:property name="body_rotation" value="1.57 0 0" />
+      <xacro:property name="body_rotation" value="1.57079632679 0 0" />
       <xacro:property name="child_translation" value="0 0 0 " />
-      <xacro:property name="child_rotation" value="3.141 0 ${mounting_rotation}" />
+      <xacro:property name="child_rotation" value="3.14159265359 0 ${mounting_rotation}" />
     </xacro:if>
     <xacro:if value="${mounting_side == 'bottom'}">
@@ -20,5 +20,5 @@
       <xacro:property name="body_rotation" value="0 0 ${mounting_rotation}" />
       <xacro:property name="child_translation" value="0 0.024 0.055" />
-      <xacro:property name="child_rotation" value="1.57 0 0" />
+      <xacro:property name="child_rotation" value="1.57079632679 0 0" />
     </xacro:if>
     <link name="${namespace}_body_link">
@@ -30,5 +30,5 @@
       <collision>
         <geometry>
-         <box size="0.055 0.055 0.078"/>
+         <box size="0.046 0.055 0.078"/>
         </geometry>
         <origin xyz="0 0.008 0.039" rpy="0 0 0" />

File: urdf/olv-xbolt.urdf (robot description, URDF)
Before this commit: robot olv-xbolt, 1 links, 0 joints
Links:
- link base_link: geometry 

File: urdf/olv-xbolt.urdf.xacro (robot description, xacro)
@@ -13,5 +13,5 @@
           <cylinder length="0.01" radius="0.022" />
         </geometry>
-        <origin rpy="0 0 0" xyz="0 0 0.005" />
+        <origin rpy="0 0 0" xyz="0 0 -0.005" />
       </collision>
     </link>

Commit message: Changed package name

File: urdf/olv-lbracket.urdf.xacro (robot description, xacro)
@@ -25,5 +25,5 @@
       <visual>
         <geometry>
-          <mesh filename="package://olive_connectors_description/meshes/olv-lbracket.dae" />
+          <mesh filename="package://olv_connector_descriptions/meshes/olv-lbracket.dae" />
         </geometry>
       </visual>

File: urdf/olv-xbolt.urdf.xacro (robot description, xacro)
@@ -5,5 +5,5 @@
       <visual>
         <geometry>
-          <mesh filename="package://olive_connectors_description/meshes/olv-xbolt.dae" />
+          <mesh filename="package://olv_connector_descriptions/meshes/olv-xbolt.dae" />
         </geometry>
         <origin rpy="0 0 0" xyz="0 0 -0.01" />

Commit message: Update.

File: urdf/olv-lbracket.urdf.xacro (robot description, xacro)
@@ -25,5 +25,5 @@
       <visual>
         <geometry>
-          <mesh filename="package://olv_connector_descriptions/meshes/olv-lbracket.dae" />
+          <mesh filename="package://olv_brackets_descriptions/meshes/olv-lbracket.dae" />
         </geometry>
       </visual>

File: urdf/olv-xbolt.urdf.xacro (robot description, xacro)
@@ -5,5 +5,5 @@
       <visual>
         <geometry>
-          <mesh filename="package://olv_connector_descriptions/meshes/olv-xbolt.dae" />
+          <mesh filename="package://olv_brackets_descriptions/meshes/olv-xbolt.dae" />
         </geometry>
         <origin rpy="0 0 0" xyz="0 0 -0.01" />
